Commit message: Fixed position and rotation of depth cameras

File: unitree_ros/robots/go1_description/xacro/depthCamera.xacro (robot description, xacro)
@@ -9,19 +9,19 @@
         <link name="camera_${name}">
             <collision>
-            <origin xyz="0 0 0" rpy="0 0 0"/>
-            <geometry>
-                <box size=".001 .001 .001"/>
-            </geometry>
+                <origin xyz="0 0 0" rpy="0 0 0"/>
+                <geometry>
+                    <box size=".001 .001 .001"/>
+                </geometry>
             </collision>
             <visual>
-            <origin xyz="0 0 0" rpy="0 0 0"/>
-            <geometry>
-                <mesh filename="package://go1_description/meshes/depthCamera.dae" scale="1 1 1"/>
-            </geometry>
+                <origin xyz="0 0 0" rpy="0 0 0"/>
+                <geometry>
+                    <mesh filename="package://go1_description/meshes/depthCamera.dae" scale="1 1 1"/>
+                </geometry>
             </visual>
             <inertial>
-            <mass value="1e-5" />
-            <origin xyz="0 0 0" rpy="0 0 0"/>
-            <inertia ixx="1e-6" ixy="0" ixz="0" iyy="1e-6" iyz="0" izz="1e-6" />
+                <mass value="1e-5" />
+                <origin xyz="0 0 0" rpy="0 0 0"/>
+                <inertia ixx="1e-6" ixy="0" ixz="0" iyy="1e-6" iyz="0" izz="1e-6" />
             </inertial>
         </link>

File: unitree_ros/robots/go1_description/xacro/robot.xacro (robot description, xacro)
@@ -89,17 +89,17 @@
     <xacro:leg name="RL" mirror="1"  mirror_dae="True"   front_hind="-1" front_hind_dae="False" />
     <xacro:depthCamera camID="1" name="face">
-        <origin rpy="${PI} 0 0" xyz="0.2785 0.0125 0.0167"/>
+        <origin rpy="0 0 0" xyz="0.2785 -0.0125 0.0167"/>
     </xacro:depthCamera>
     <xacro:depthCamera camID="2" name="chin">
-        <origin rpy="${PI} ${PI/2} 0" xyz="0.2522 0.0125 -0.0436"/>
+        <origin rpy="0 ${PI/2} 0" xyz="0.2522 -0.0125 -0.0436"/>
     </xacro:depthCamera>
     <xacro:depthCamera camID="3" name="left">
-        <origin rpy="${PI} 0.2618 ${PI/2}" xyz="-0.066 0.082 -0.0176"/>
+        <origin rpy="0 0.2618 ${PI/2}" xyz="-0.041 0.082 -0.0176"/>
     </xacro:depthCamera>
     <xacro:depthCamera camID="4" name="right">
-        <origin rpy="${PI} 0.2618 ${-PI/2}" xyz="-0.041 -0.082 -0.0176"/>
+        <origin rpy="0 0.2618 ${-PI/2}" xyz="-0.066 -0.082 -0.0176"/>
     </xacro:depthCamera>
     <xacro:depthCamera camID="5" name="rearDown">
-        <origin rpy="${PI} ${PI/2} 0" xyz="-0.0825 0.0125 -0.04365"/>
+        <origin rpy="0 ${PI/2} 0" xyz="-0.0825 -0.0125 -0.04365"/>
     </xacro:depthCamera>
     <joint name="camera_laserscan_joint_left" type="fixed">
