Commit message: Fixed lidar settings

File: unitree_ros/robots/go1_description/xacro/lidar.xacro (robot description, xacro)
@@ -1,11 +1,19 @@
 <?xml version="1.0"?>
-<robot xmlns:xacro="http://www.ros.org/wiki/xacro" >
+<robot xmlns:xacro="http://www.ros.org/wiki/xacro" name="hokuyo">
+<xacro:macro name="lidar" params="parent *origin">
     <joint name="laser_joint" type="fixed">
-        <parent link="trunk"/>
-        <child link="laser_frame"/>
-        <origin xyz="0.05 0 0.08" rpy="0 0 0"/>
+        <xacro:insert_block name="origin"/>
+        <parent link="${parent}"/>
+        <child link="laser_link"/>
     </joint>
-    <link name="laser_frame">
+    <link name="laser_link">
+        <collision>
+            <origin xyz="0 0 0" rpy="0 0 0"/>
+            <geometry>
+                <cylinder radius="0.05" length="0.05"/>
+            </geometry>
+        </collision>
         <visual>
+            <origin xyz="0 0 0" rpy="0 0 0"/>
             <geometry>
                 <cylinder radius="0.05" length="0.05"/>
@@ -13,40 +21,44 @@
             <material name="black"/>
         </visual>
-        <collision>
-            <geometry>
-                <cylinder radius="0.05" length="0.04"/>
-            </geometry>
-        </collision>
         <inertial>
-            <mass value="0.1" />
-            <inertia ixx="0.001" ixy="0.0" ixz="0.0"
-                iyy="0.001" iyz="0.0"
-                izz="0.001" />
+            <mass value="1e-5" />
+            <origin xyz="0 0 0" rpy="0 0 0"/>
+            <inertia ixx="1e-6" ixy="0" ixz="0" iyy="1e-6" iyz="0" izz="1e-6" />
         </inertial>
     </link>
-    <gazebo reference="laser_frame">
+    <gazebo reference="laser_link">
         <material>Gazebo/Black</material>
-        <sensor name="laser" type="ray">
-            <pose> 0 0 0 0 0 0 </pose>
+        <gravity>true</gravity>
+        <sensor type="ray" name="laser">
+            <pose>0 0 0 0 0 0</pose>
             <visualize>false</visualize>
-            <update_rate>10</update_rate>
+            <update_rate>40</update_rate>
             <ray>
                 <scan>
                     <horizontal>
                         <samples>360</samples>
-                        <min_angle>-3.14</min_angle>
-                        <max_angle>3.14</max_angle>
+                        <resolution>1</resolution>
+                        <min_angle>${-pi}</min_angle>
+                        <max_angle>${pi}</max_angle>
                     </horizontal>
                 </scan>
                 <range>
-                    <min>0.3</min>
-                    <max>12</max>
+                    <min>0.2</min>
+                    <max>40</max>
+                    <resolution>0.025</resolution>
                 </range>
+                <noise>
+                    <type>gaussian</type>
+                    <mean>0.0</mean>
+                    <stddev>0.0</stddev>
+                </noise>
             </ray>
             <plugin name="laser_controller" filename="libgazebo_ros_laser.so">
-                <topicName>/scan</topicName>
-                <frame_name>laser_frame</frame_name>
+                <robotNamespace></robotNamespace>
+                <topicName>scan</topicName>
+                <frameName>laser_link</frameName>
             </plugin>
         </sensor>
     </gazebo>
+</xacro:macro>
 </robot>

File: unitree_ros/robots/go1_description/xacro/robot.xacro (robot description, xacro)
@@ -126,3 +126,6 @@
         <origin rpy="0 0 0" xyz="0.2747 0.0 -0.0088"/>
     </xacro:ultraSound>
+    <xacro:lidar parent="trunk">
+        <origin rpy="0 0 0" xyz="0.05 0 0.08"/>
+    </xacro:lidar>
 </robot>
