Commit message: Updated urdf

File: unitree_ros/robots/go1_description/urdf/go1.urdf (robot description, URDF)
Before this commit: robot go1, 46 links, 45 joints
Links:
- added link laser_link, mass 1e-5; collision cylinder length=0.05 radius=0.05; visual cylinder length=0.05 radius=0.05
- link FL_calf_rotor: geometry visual cylinder length=0.02 radius=0.035
- link FL_hip_rotor: geometry visual cylinder length=0.02 radius=0.035
- link FL_thigh_rotor: geometry visual cylinder length=0.02 radius=0.035
- link FR_calf_rotor: geometry visual cylinder length=0.02 radius=0.035
- link FR_hip_rotor: geometry visual cylinder length=0.02 radius=0.035
- link FR_thigh_rotor: geometry visual cylinder length=0.02 radius=0.035
- link RL_calf_rotor: geometry visual cylinder length=0.02 radius=0.035
- link RL_hip_rotor: geometry visual cylinder length=0.02 radius=0.035
- link RL_thigh_rotor: geometry visual cylinder length=0.02 radius=0.035
- link RR_calf_rotor: geometry visual cylinder length=0.02 radius=0.035
- link RR_hip_rotor: geometry visual cylinder length=0.02 radius=0.035
- link RR_thigh_rotor: geometry visual cylinder length=0.02 radius=0.035
Joints:
- added joint laser_joint: type fixed, parent trunk, child laser_link, origin xyz=0.05 0 0.08 rpy=0 0 0
- joint camera_joint_chin: origin xyz=0.2522 0.0125 -0.0436 rpy=3.141592653589793 1.5707963267948966 0 -> xyz=0.2522 -0.0125 -0.0436 rpy=0 1.5707963267948966 0
- joint camera_joint_face: origin xyz=0.2785 0.0125 0.0167 rpy=3.141592653589793 0 0 -> xyz=0.2785 -0.0125 0.0167 rpy=0 0 0
- joint camera_joint_left: origin xyz=-0.066 0.082 -0.0176 rpy=3.141592653589793 0.2618 1.5707963267948966 -> xyz=-0.041 0.082 -0.0176 rpy=0 0.2618 1.5707963267948966
- joint camera_joint_rearDown: origin xyz=-0.0825 0.0125 -0.04365 rpy=3.141592653589793 1.5707963267948966 0 -> xyz=-0.0825 -0.0125 -0.04365 rpy=0 1.5707963267948966 0
- joint camera_joint_right: origin xyz=-0.041 -0.082 -0.0176 rpy=3.141592653589793 0.2618 -1.5707963267948966 -> xyz=-0.066 -0.082 -0.0176 rpy=0 0.2618 -1.5707963267948966
