Commit message: Fixed Z1 urdf

File: unitree_ros/robots/z1_description/xacro/robot.xacro (robot description, xacro)
@@ -48,10 +48,4 @@
             </geometry>
         </visual>
-        <!-- <collision>
-            <geometry>
-                <cylinder length="${2*motor_height}" radius="${motor_diameter}"/>
-            </geometry>
-            <origin rpy="0 0 0" xyz="0 0 0"/>
-        </collision> -->
         <inertial>
             <origin rpy="0 0 0" xyz="${L01_ComX} ${L01_ComY} ${L01_ComZ}"/>
@@ -130,5 +124,5 @@
                 <cylinder length="0.059" radius="${motor_diameter}"/>
             </geometry>
-            <origin rpy="0 ${PI/2.0} 0" xyz="${0.065+0.185-0.059/2.0} 0 0.055"/>
+            <origin rpy="0 ${PI/2.0} ${PI/2.0}" xyz="${0.065+0.185-0.059/2.0} 0 0.055"/>
         </collision>
         <inertial>
@@ -158,7 +152,7 @@
         <collision>
             <geometry>
-                <cylinder length="0.073" radius="${motor_diameter}"/>
-            </geometry>
-            <origin rpy="${PI/2.0} 0 0" xyz="0.0472 0 0"/>
+                <cylinder length="${motor_height + 2*0.008}" radius="${motor_diameter}"/>
+            </geometry>
+            <origin rpy="${0 0 0" xyz="0.072 0 0"/>
         </collision>
         <inertial>

File: unitree_ros/robots/z1_description/xacro/z1.urdf (robot description, URDF)
Before this commit: robot z1_description, 8 links, 7 joints
Links:
- link link00: geometry collision cylinder length=0.051 radius=0.0325; visual mesh filename=package://z1_description/meshes/visual/z1_Link00.dae scale=1 1 1
- link link01: geometry visual mesh filename=package://z1_description/meshes/visual/z1_Link01.dae scale=1 1 1
- link link02: geometry collision cylinder length=0.051 radius=0.0325; collision cylinder length=0.102 radius=0.0325
- link link03: geometry collision cylinder length=0.059 radius=0.0325; collision cylinder length=0.116 radius=0.02
- link link04: geometry collision cylinder length=0.067 radius=0.0325; visual mesh filename=package://z1_description/meshes/visual/z1_Link04.dae scale=1 1 1
- link link05: geometry visual mesh filename=package://z1_description/meshes/visual/z1_Link05.dae scale=1 1 1
- link link06: geometry collision cylinder length=0.051 radius=0.0325; visual mesh filename=package://z1_description/meshes/visual/z1_Link06.dae scale=1 1 1
Joints:
- joint joint1: limit lower=-2.6179938779914944 upper=2.6179938779914944 effort=30.0 velocity=10 -> lower=-2.6179938779914944 upper=2.6179938779914944 effort=30.0 velocity=3.1415
- joint joint2: limit lower=0.0 upper=3.141592653589793 effort=60.0 velocity=10 -> lower=0.0 upper=2.9670597283903604 effort=60.0 velocity=3.1415
- joint joint3: limit lower=-4.782202150464463 upper=0.0 effort=30.0 velocity=10 -> lower=-2.8797932657906435 upper=0.0 effort=30.0 velocity=3.1415
- joint joint4: limit lower=-1.7453292519943295 upper=1.5707963267948966 effort=30.0 velocity=10 -> lower=-1.5184364492350666 upper=1.5184364492350666 effort=30.0 velocity=3.1415
- joint joint5: limit lower=-1.7278759594743864 upper=1.7278759594743864 effort=30.0 velocity=10 -> lower=-1.3439035240356338 upper=1.3439035240356338 effort=30.0 velocity=3.1415
- joint joint6: limit lower=-2.792526803190927 upper=2.792526803190927 effort=30.0 velocity=10 -> lower=-2.792526803190927 upper=2.792526803190927 effort=30.0 velocity=3.1415
